Commit message: add some templates

File: nasa_r2_common/r2_description/robots/r2.display.urdf.xacro (robot description, xacro)
@@ -1,8 +1,8 @@
 <?xml version="1.0" ?>
 <robot name="r2" xmlns:controller="http://playerstage.sourceforge.net/gazebo/xmlschema/#controller"
-			xmlns:interface="http://www.ros.org/wiki/xacro"
+			xmlns:interface="http://playerstage.sourceforge.net/gazebo/xmlschema/#interface"
 			xmlns:sensor="http://playerstage.sourceforge.net/gazebo/xmlschema/#sensor"
-			xmlns:xacro="http://www.ros.org/wiki/xacro">
-  <xacro:property name="robot_name" value= "r2/" />
+			xmlns:xacro="http://playerstage.sourceforge.net/gazebo/xmlschema/#interface">
+  <property name="robot_name" value= "r2/" />
   <xacro:include filename="$(find r2_description)/robots/r2.urdf.xacro" />
   <xacro:include filename="$(find r2_description)/urdf/r2.gazebo.xacro" />

File: nasa_r2_common/r2_description/robots/r2.sim.urdf.xacro (robot description, xacro)
@@ -1,8 +1,8 @@
 <?xml version="1.0" ?>
 <robot name="r2" xmlns:controller="http://playerstage.sourceforge.net/gazebo/xmlschema/#controller"
-			xmlns:interface="http://www.ros.org/wiki/xacro"
+			xmlns:interface="http://playerstage.sourceforge.net/gazebo/xmlschema/#interface"
 			xmlns:sensor="http://playerstage.sourceforge.net/gazebo/xmlschema/#sensor"
-			xmlns:xacro="http://www.ros.org/wiki/xacro">
-  <xacro:property name="robot_name" value= "r2/" />
+			xmlns:xacro="http://playerstage.sourceforge.net/gazebo/xmlschema/#interface">
+  <property name="robot_name" value= "r2/" />
   <xacro:include filename="$(find r2_description)/robots/r2.urdf.xacro" />
   <xacro:include filename="$(find r2_description)/urdf/r2.gazebo.xacro" />

File: nasa_r2_common/r2_description/robots/r2.urdf.xacro (robot description, xacro)
@@ -1,8 +1,8 @@
 <?xml version="1.0" ?>
 <robot name="r2" xmlns:controller="http://playerstage.sourceforge.net/gazebo/xmlschema/#controller"
-			xmlns:interface="http://www.ros.org/wiki/xacro"
+			xmlns:interface="http://playerstage.sourceforge.net/gazebo/xmlschema/#interface"
 			xmlns:sensor="http://playerstage.sourceforge.net/gazebo/xmlschema/#sensor"
-			xmlns:xacro="http://www.ros.org/wiki/xacro">
-  <xacro:property name="robot_name" value= "r2/" />
+			xmlns:xacro="http://playerstage.sourceforge.net/gazebo/xmlschema/#interface">
+  <property name="robot_name" value= "r2/" />
   <xacro:include filename="$(find r2_description)/urdf/r2.common.xacro" />
   <xacro:include filename="$(find r2_description)/urdf/r2.base.xacro" />

File: nasa_r2_common/r2_description/robots/r2_fullbody.urdf.xacro (robot description, xacro)
@@ -2,9 +2,9 @@
   <robot xmlns:sensor="http://playerstage.sourceforge.net/gazebo/xmlschema/#sensor"
        xmlns:controller="http://playerstage.sourceforge.net/gazebo/xmlschema/#controller"
-       xmlns:interface="http://www.ros.org/wiki/xacro"
-       xmlns:xacro="http://www.ros.org/wiki/xacro"
+       xmlns:interface="http://playerstage.sourceforge.net/gazebo/xmlschema/#interface"
+       xmlns:xacro="http://playerstage.sourceforge.net/gazebo/xmlschema/#interface"
        name="r2_fullbody" >
   <link name="world"/>
-  <xacro:property name="robot_name" value= "r2/" />
+  <property name="robot_name" value= "r2/" />
 <!--  transforms in first joint don't seem to work properly-->
   <joint name="${robot_name}fixed/world/robot_world" type="fixed">

File: nasa_r2_common/r2_description/robots/r2_fullbody_no_world.urdf.xacro (robot description, xacro)
@@ -1,5 +1,5 @@
 <?xml version="1.0" ?>
-<robot name="r2" xmlns:xacro="http://www.ros.org/wiki/xacro">
-  <xacro:property name="robot_name" value= "r2/" />
+<robot name="r2" xmlns:xacro="http://playerstage.sourceforge.net/gazebo/xmlschema/#interface">
+  <property name="robot_name" value= "r2/" />
   <link name="${robot_name}robot_world"/>
   <joint name="${robot_name}fixed/robot_world/robot_base" type="fixed">

File: nasa_r2_common/r2_description/robots/r2_legs.urdf.xacro (robot description, xacro)
@@ -1,8 +1,8 @@
 <?xml version="1.0" ?>
 <robot name="r2" xmlns:controller="http://playerstage.sourceforge.net/gazebo/xmlschema/#controller"
-                 xmlns:interface="http://www.ros.org/wiki/xacro"
+                 xmlns:interface="http://playerstage.sourceforge.net/gazebo/xmlschema/#interface"
                  xmlns:sensor="http://playerstage.sourceforge.net/gazebo/xmlschema/#sensor"
-                 xmlns:xacro="http://www.ros.org/wiki/xacro">
-  <xacro:property name="robot_name" value= "r2/" />
+                 xmlns:xacro="http://playerstage.sourceforge.net/gazebo/xmlschema/#interface">
+  <property name="robot_name" value= "r2/" />
   <xacro:include filename="$(find r2_description)/urdf/r2.common.xacro" />
   <xacro:include filename="$(find r2_description)/urdf/r2_legs/r2_legs.stand.xacro" />

File: nasa_r2_common/r2_description/robots/r2_orocos.sim.urdf.xacro (robot description, xacro)
@@ -1,8 +1,8 @@
 <?xml version="1.0" ?>
 <robot name="r2_orocos" xmlns:controller="http://playerstage.sourceforge.net/gazebo/xmlschema/#controller"
-			xmlns:interface="http://www.ros.org/wiki/xacro"
+			xmlns:interface="http://playerstage.sourceforge.net/gazebo/xmlschema/#interface"
 			xmlns:sensor="http://playerstage.sourceforge.net/gazebo/xmlschema/#sensor"
-			xmlns:xacro="http://www.ros.org/wiki/xacro">
-  <xacro:property name="robot_name" value= "r2/" />
+			xmlns:xacro="http://playerstage.sourceforge.net/gazebo/xmlschema/#interface">
+  <property name="robot_name" value= "r2/" />
   <xacro:include filename="$(find r2_description)/urdf/models/r2c_upper_body.urdf.xacro" />
   <xacro:include filename="$(find r2_description)/urdf/r2.gazebo.xacro" />

File: nasa_r2_common/r2_description/robots/r2c_full_body.sim.urdf.xacro (robot description, xacro)
@@ -1,8 +1,8 @@
 <?xml version="1.0" ?>
 <robot name="r2c_full_body" xmlns:controller="http://playerstage.sourceforge.net/gazebo/xmlschema/#controller"
-			xmlns:interface="http://www.ros.org/wiki/xacro"
+			xmlns:interface="http://playerstage.sourceforge.net/gazebo/xmlschema/#interface"
 			xmlns:sensor="http://playerstage.sourceforge.net/gazebo/xmlschema/#sensor"
-			xmlns:xacro="http://www.ros.org/wiki/xacro">
-  <xacro:property name="robot_name" value= "r2/" />
+			xmlns:xacro="http://playerstage.sourceforge.net/gazebo/xmlschema/#interface">
+  <property name="robot_name" value= "r2/" />
   <link name="world"/>
   <!--  transforms in first joint don't seem to work properly-->

File: nasa_r2_common/r2_description/robots/r2c_full_body_ISS.sim.urdf.xacro (robot description, xacro)
@@ -1,8 +1,8 @@
 <?xml version="1.0" ?>
 <robot name="r2c_full_body" xmlns:controller="http://playerstage.sourceforge.net/gazebo/xmlschema/#controller"
-			xmlns:interface="http://www.ros.org/wiki/xacro"
+			xmlns:interface="http://playerstage.sourceforge.net/gazebo/xmlschema/#interface"
 			xmlns:sensor="http://playerstage.sourceforge.net/gazebo/xmlschema/#sensor"
-			xmlns:xacro="http://www.ros.org/wiki/xacro">
-  <xacro:property name="robot_name" value= "r2/" />
+			xmlns:xacro="http://playerstage.sourceforge.net/gazebo/xmlschema/#interface">
+  <property name="robot_name" value= "r2/" />
   <xacro:include filename="$(find r2_description)/urdf/models/r2c_full_body_no_world.urdf.xacro" />
   <xacro:robot_world_origin>

File: nasa_r2_common/r2_description/robots/r2c_legs.display.urdf.xacro (robot description, xacro)
@@ -1,8 +1,8 @@
 <?xml version="1.0" ?>
 <robot name="r2c_legs" xmlns:controller="http://playerstage.sourceforge.net/gazebo/xmlschema/#controller"
-			xmlns:interface="http://www.ros.org/wiki/xacro"
+			xmlns:interface="http://playerstage.sourceforge.net/gazebo/xmlschema/#interface"
 			xmlns:sensor="http://playerstage.sourceforge.net/gazebo/xmlschema/#sensor"
-			xmlns:xacro="http://www.ros.org/wiki/xacro">
-  <xacro:property name="robot_name" value= "r2/" />
+			xmlns:xacro="http://playerstage.sourceforge.net/gazebo/xmlschema/#interface">
+  <property name="robot_name" value= "r2/" />
   <xacro:include filename="$(find r2_description/urdf/models/r2c_legs.urdf.xacro" />
   <xacro:include filename="$(find r2_description/urdf/r2c_legs.gazebo.xacro" />

File: nasa_r2_common/r2_description/robots/r2c_legs.sim.urdf.xacro (robot description, xacro)
@@ -1,8 +1,8 @@
 <?xml version="1.0" ?>
 <robot name="r2c_legs" xmlns:controller="http://playerstage.sourceforge.net/gazebo/xmlschema/#controller"
-			xmlns:interface="http://www.ros.org/wiki/xacro"
+			xmlns:interface="http://playerstage.sourceforge.net/gazebo/xmlschema/#interface"
 			xmlns:sensor="http://playerstage.sourceforge.net/gazebo/xmlschema/#sensor"
-			xmlns:xacro="http://www.ros.org/wiki/xacro">
-  <xacro:property name="robot_name" value= "r2/" />
+			xmlns:xacro="http://playerstage.sourceforge.net/gazebo/xmlschema/#interface">
+  <property name="robot_name" value= "r2/" />
   <xacro:include filename="$(find r2_description)/urdf/models/r2c_legs.urdf.xacro" />
   <xacro:include filename="$(find r2_description)/urdf/r2c_legs.gazebo.xacro" />

File: nasa_r2_common/r2_description/robots/r2c_legs_control.urdf.xacro (robot description, xacro)
@@ -1,8 +1,8 @@
 <?xml version="1.0" ?>
 <robot name="r2c_legs" xmlns:controller="http://playerstage.sourceforge.net/gazebo/xmlschema/#controller"
-                       xmlns:interface="http://www.ros.org/wiki/xacro"
+                       xmlns:interface="http://playerstage.sourceforge.net/gazebo/xmlschema/#interface"
                        xmlns:sensor="http://playerstage.sourceforge.net/gazebo/xmlschema/#sensor"
-                       xmlns:xacro="http://www.ros.org/wiki/xacro">
-  <xacro:property name="robot_name" value= "r2/" />
+                       xmlns:xacro="http://playerstage.sourceforge.net/gazebo/xmlschema/#interface">
+  <property name="robot_name" value= "r2/" />
   <link name="${robot_name}robot_world"/>
   <non_visual_link name="${robot_name}robot_base"/>

File: nasa_r2_common/r2_description/robots/r2c_torso.sim.urdf.xacro (robot description, xacro)
@@ -1,8 +1,8 @@
 <?xml version="1.0" ?>
 <robot name="r2_torso" xmlns:controller="http://playerstage.sourceforge.net/gazebo/xmlschema/#controller"
-			xmlns:interface="http://www.ros.org/wiki/xacro"
+			xmlns:interface="http://playerstage.sourceforge.net/gazebo/xmlschema/#interface"
 			xmlns:sensor="http://playerstage.sourceforge.net/gazebo/xmlschema/#sensor"
-			xmlns:xacro="http://www.ros.org/wiki/xacro">
-  <xacro:property name="robot_name" value= "r2/" />
+			xmlns:xacro="http://playerstage.sourceforge.net/gazebo/xmlschema/#interface">
+  <property name="robot_name" value= "r2/" />
   <xacro:include filename="$(find r2_description)/urdf/models/r2c_upper_body_stand.urdf.xacro" />
   <xacro:include filename="$(find r2_description)/urdf/r2.gazebo.xacro" />

File: nasa_r2_common/r2_description/urdf/gazebo_plugins/gazebo_interface.xacro (robot description, xacro)
@@ -1,7 +1,7 @@
 <?xml version="1.0"?>
 <robot name="r2_c_full_body" xmlns:controller="http://playerstage.sourceforge.net/gazebo/xmlschema/#controller"
-			xmlns:interface="http://www.ros.org/wiki/xacro"
+			xmlns:interface="http://playerstage.sourceforge.net/gazebo/xmlschema/#interface"
 			xmlns:sensor="http://playerstage.sourceforge.net/gazebo/xmlschema/#sensor"
-			xmlns:xacro="http://www.ros.org/wiki/xacro">
+			xmlns:xacro="http://playerstage.sourceforge.net/gazebo/xmlschema/#interface">
   <gazebo>
     <controller:gazebo_interface name="gazebo_interface" plugin="libgazebo_interface.so">

File: nasa_r2_common/r2_description/urdf/gazebo_plugins/leg_grippers.xacro (robot description, xacro)
@@ -1,7 +1,7 @@
 <?xml version="1.0"?>
 <robot name="r2_c_full_body" xmlns:controller="http://playerstage.sourceforge.net/gazebo/xmlschema/#controller"
-			xmlns:interface="http://www.ros.org/wiki/xacro"
+			xmlns:interface="http://playerstage.sourceforge.net/gazebo/xmlschema/#interface"
 			xmlns:sensor="http://playerstage.sourceforge.net/gazebo/xmlschema/#sensor"
-			xmlns:xacro="http://www.ros.org/wiki/xacro">
+			xmlns:xacro="http://playerstage.sourceforge.net/gazebo/xmlschema/#interface">
   <gazebo>
     <controller:gazebo_gripper name="left_gazebo_gripper" plugin="libgazebo_gripper.so">

File: nasa_r2_common/r2_description/urdf/gazebo_plugins/p3d_base_controller.xacro (robot description, xacro)
@@ -1,7 +1,7 @@
 <?xml version="1.0"?>
 <robot name="r2_c_full_body" xmlns:controller="http://playerstage.sourceforge.net/gazebo/xmlschema/#controller"
-			xmlns:interface="http://www.ros.org/wiki/xacro"
+			xmlns:interface="http://playerstage.sourceforge.net/gazebo/xmlschema/#interface"
 			xmlns:sensor="http://playerstage.sourceforge.net/gazebo/xmlschema/#sensor"
-			xmlns:xacro="http://www.ros.org/wiki/xacro">
+			xmlns:xacro="http://playerstage.sourceforge.net/gazebo/xmlschema/#interface">
   <gazebo>
     <controller:gazebo_ros_p3d name="p3d_base_controller" plugin="libgazebo_ros_p3d.so">

File: nasa_r2_common/r2_description/urdf/gazebo_plugins/r2.gazebo.controller.xacro (robot description, xacro)
@@ -1,7 +1,7 @@
 <?xml version="1.0"?>
 <robot xmlns:controller="http://playerstage.sourceforge.net/gazebo/xmlschema/#controller"
-			xmlns:interface="http://www.ros.org/wiki/xacro"
+			xmlns:interface="http://playerstage.sourceforge.net/gazebo/xmlschema/#interface"
 			xmlns:sensor="http://playerstage.sourceforge.net/gazebo/xmlschema/#sensor"
-			xmlns:xacro="http://www.ros.org/wiki/xacro">
+			xmlns:xacro="http://playerstage.sourceforge.net/gazebo/xmlschema/#interface">
   <gazebo>
     <controller:gazebo_ros_controller_manager name="gazebo_ros_controller_manager" plugin="libgazebo_ros_controller_manager.so">

File: nasa_r2_common/r2_description/urdf/gazebo_plugins/r2.transmissions.xacro (robot description, xacro)
@@ -1,6 +1,6 @@
 <?xml version="1.0"?>
-<robot xmlns:xacro="http://www.ros.org/wiki/xacro">
+<robot>
   <!-- transmission xacro -->
-  <xacro:macro name="r2_trans" params="part joint reduction tc">
+  <macro name="r2_trans" params="part joint reduction tc">
      <transmission name="${part}_j${joint}_trans" type="pr2_mechanism_model/SimpleTransmission">
        <actuator name="${part}_j${joint}_motor"/>
@@ -9,7 +9,7 @@
        <motorTorqueConstant>${tc}</motorTorqueConstant>
      </transmission>
-  </xacro:macro>
+  </macro>
   <!-- r2_arm_transmission xacro -->
-  <xacro:macro name="r2_arm_trans" params="side">
+  <macro name="r2_arm_trans" params="side">
      <r2_trans part="${side}" joint="0" reduction="160" tc="0.305"/>
      <r2_trans part="${side}" joint="1" reduction="160" tc="0.305"/>
@@ -37,5 +37,5 @@
      <r2_trans part="${side}/hand/little" joint="1" reduction="1" tc="1"/>
      <r2_trans part="${side}/hand/little" joint="2" reduction="1" tc="1"/>
-  </xacro:macro>
+  </macro>
   <r2_trans part="${robot_name}waist" joint="0" reduction="0.00625" tc="0.1"/>
   <r2_arm_trans side="${robot_name}left_arm"/>

File: nasa_r2_common/r2_description/urdf/gazebo_plugins/taskboard.panel_a.controller.xacro (robot description, xacro)
@@ -1,7 +1,7 @@
 <?xml version="1.0"?>
 <robot name="panel_a" xmlns:controller="http://playerstage.sourceforge.net/gazebo/xmlschema/#controller"
-			xmlns:interface="http://www.ros.org/wiki/xacro"
+			xmlns:interface="http://playerstage.sourceforge.net/gazebo/xmlschema/#interface"
 			xmlns:sensor="http://playerstage.sourceforge.net/gazebo/xmlschema/#sensor"
-			xmlns:xacro="http://www.ros.org/wiki/xacro">
+			xmlns:xacro="http://playerstage.sourceforge.net/gazebo/xmlschema/#interface">
   <gazebo>
     <controller:panel_a_interface name="panel_a_interface" plugin="libgazebo_taskboard.so">

File: nasa_r2_common/r2_description/urdf/models/r2.base.xacro (robot description, xacro)
@@ -1,4 +1,4 @@
 <?xml version="1.0"?>
-<robot xmlns:xacro="http://www.ros.org/wiki/xacro">
+<robot>
   <link name="world"/>
   <joint name="${robot_name}fixed/world/robot_world" type="fixed">
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